File: controller/_autosave-silver-platter.kicad_sch (KiCad schematic)
At the start: 64 parts, among them J1 UART, J11 LED1_B, J12 LED1_G, J13 LED1_R, J14 LED_ANODE, J15 LED2_B, J16 LED2_G, J17 LED2_R, J19 RX_VDD, J2 JTAG/SWJ, J20 RX_iBUS, J21 RX_GND, J22 BOOT, J23 +BATT, J24 -BATT, J3 VDD_ACC, J4 SCL_ACC, J5 SDA_ACC, J6 GND_ACC, J8 CH1_ESC, J9 CH2_ESC, Q1 Q_NMOS, Q2 Q_NMOS, Q3 Q_NMOS, SW1 SW_Push, U1 STM32F205RETx, U2 TLV74033PDBVR, U3 LMR50410Y5FQDBVRQ1

Commit message: Layout draft 1
Parts:
- removed TP1: +5V, TestPoint:TestPoint_Plated_Hole_D2.0mm, symbol Connector:TestPoint
- removed TP2: +3V3, TestPoint:TestPoint_Plated_Hole_D2.0mm, symbol Connector:TestPoint
- removed TP3: +BATT, TestPoint:TestPoint_Plated_Hole_D2.0mm, symbol Connector:TestPoint
