File: controller/silver-platter.kicad_pcb (KiCad board)
At the start: 2 copper layers, 67 parts, among them J1 UART, J10 GND_ESC, J11 LED1_B, J12 LED1_G, J13 LED1_R, J14 LED1_ANODE, J15 LED2_B, J16 LED2_G, J17 LED2_R, J18 LED2_ANODE, J19 RX_VDD, J2 JTAG/SWJ, J20 RX_iBUS, J21 RX_GND, J22 BOOT, J23 +BATT, J24 -BATT, J3 VDD_ACCEL, J4 SCL_ACCEL, J5 SDA_ACCEL, J6 GND_ACCEL, J7 VBAT_ESC, J8 CH1_ESC, J9 CH2_ESC, Q1 Q_NMOS, Q2 Q_NMOS, Q3 Q_NMOS, SW1 SW_Push, U1 STM32F205RETx, U2 TLV74033PDBVR, U3 LMR50410Y5FQDBVRQ1

Commit message: Layout draft 1
Parts:
- removed J10: GND_ESC, TestPoint:TestPoint_Pad_4.0x4.0mm
- removed J18: LED2_ANODE, TestPoint:TestPoint_Pad_4.0x4.0mm
- removed J7: VBAT_ESC, TestPoint:TestPoint_Pad_4.0x4.0mm
- removed TP1: +5V, TestPoint:TestPoint_Plated_Hole_D2.0mm
- removed TP2: +3V3, TestPoint:TestPoint_Plated_Hole_D2.0mm
- removed TP3: +BATT, TestPoint:TestPoint_Plated_Hole_D2.0mm
- J14: value LED1_ANODE -> LED_ANODE
- J20: value RX_iBUS -> iBUS
- J21: value RX_GND -> GND
- J3: value VDD_ACCEL -> VDD_ACC
- J4: value SCL_ACCEL -> SCL_ACC
- J5: value SDA_ACCEL -> SDA_ACC
- J6: value GND_ACCEL -> GND_ACC
- moved J2 174.1 mm to (181.0, 103.5), turned to -90 degrees
- moved J8 173.0 mm to (167.6, 121.9)
- moved J9 164.4 mm to (161.3, 121.9)
- moved J14 161.8 mm to (184.2, 77.5)
- moved J6 155.8 mm to (152.4, 121.9)
- moved J5 153.4 mm to (146.1, 121.9)
- moved J4 151.4 mm to (139.7, 121.9)
- moved J1 151.2 mm to (175.3, 121.9), turned to 90 degrees
- moved J17 150.5 mm to (176.5, 77.5)
- moved J13 150.3 mm to (170.2, 77.5)
- moved J3 150.0 mm to (133.3, 121.9)
- moved C2 145.7 mm to (158.5, 113.0)
- moved C10 140.1 mm to (154.8, 114.6), turned to 180 degrees
- moved R4 139.7 mm to (171.3, 102.6), turned to 180 degrees
- moved D2 139.7 mm to (167.5, 102.6), turned to 180 degrees
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Connections:
- Q1 pad 1: (no net) -> /LED_R_PWM
- Q1 pad 2: (no net) -> GND
- Q1 pad 3: (no net) -> Net-(Q1-D)
- Q2 pad 1: (no net) -> /LED_G_PWM
- Q2 pad 2: (no net) -> GND
- Q2 pad 3: (no net) -> Net-(Q2-D)
- Q3 pad 1: (no net) -> /LED_B_PWM
- Q3 pad 2: (no net) -> GND
- Q3 pad 3: (no net) -> Net-(Q3-D)
- R10 pad 2: Net-(Q1-PadD) -> Net-(Q1-D)
- R5 pad 1: Net-(Q1-PadD) -> Net-(Q1-D)
- R6 pad 1: Net-(Q2-PadD) -> Net-(Q2-D)
- R7 pad 1: Net-(Q3-PadD) -> Net-(Q3-D)
- R8 pad 2: Net-(Q3-PadD) -> Net-(Q3-D)
- R9 pad 2: Net-(Q2-PadD) -> Net-(Q2-D)
- U2 pad 4: unconnected-(U2-NC-Pad4) -> GND
Routing:
- net /NRST: track 0.00 -> 58.2 mm, vias 0 -> 2
- net /USART1_RX: track 0.00 -> 40.2 mm
- net +BATT: track 0.00 -> 35.5 mm
- net /JTMS_SWDIO: track 0.00 -> 33.9 mm
- net /USART1_TX: track 0.00 -> 33.2 mm, vias 0 -> 2
- net /nJTRST: track 0.00 -> 30.9 mm
- net /JTDO_SWO: track 0.00 -> 30.3 mm, vias 0 -> 2
- net /JTCK_SWCLK: track 0.00 -> 29.3 mm
- net /JTDI: track 0.00 -> 29.2 mm
- net /iBUS: track 0.00 -> 27.5 mm
- net /DSHOT_CH1: track 0.00 -> 20.0 mm
- net /I2C2_SCL: track 0.00 -> 19.4 mm
- net Net-(Q1-D): track 0.00 -> 17.5 mm
- net Net-(U1-PA1): track 0.00 -> 16.9 mm
- net /BOOT: track 0.00 -> 16.7 mm
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- added copper zone on In2.Cu, net +3V3
- added copper zone on F.Cu, net +5V
- added copper zone on In2.Cu, net +5V
- added copper zone on F.Cu, net +BATT
- added copper zone on F.Cu, net GND
- added copper zone on In1.Cu, net GND
- added copper zone on F.Cu, net Net-(U3-SW)
Other:
- board outline added: 69.9 x 54 mm
- copper layers 2 -> 4
- board text added: "+"
- board text added: "+3V3"
- board text added: "+5V"
- board text added: "-"
- board text added: "Accelerometer"
- board text added: "B"
- board text added: "CH1"
- board text added: "CH2"
- board text added: "DShot ESC"
- board text added: "G"
- board text added: "GND"
- board text added: "PWR"
- board text added: "R"
- board text added: "RESET"
- board text added: "RGB LED"
- board text added: "RX"
- board text added: "Receiver"
- board text added: "SCL"
- board text added: "SDA"
- board text added: "TX"

Commit message: Silkscreen
Other:
- board text added: "Meltybrain Control Board v1.0"
Changed lines of the file:
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@@
+	)
+	(gr_line
+		(start 165.862 101.6)
+		(end 162.56 101.6)
+		(stroke
+			(width 0.153)
+			(type solid)
+		)
+		(layer "F.SilkS")
+	)
+	(gr_rect
+		(start 119.38 91.44)
+		(end 132.08 97.79)
+		(stroke
+			(width 0.1)
+			(type dash)
+		)
+		(fill no)
+		(layer "F.SilkS")
 	)
 	(gr_line
@@
 	)
 	(gr_line
+		(start 162.56 98.298)
+		(end 162.56 100.33)
+		(stroke
+			(width 0.153)
+			(type solid)
+		)
+		(layer "F.SilkS")
+	)
+	(gr_line
 		(start 130.175 118.11)
 		(end 155.575 118.11)
@@
 	)
 	(gr_line
+		(start 162.56 94.996)
+		(end 162.56 97.028)
+		(stroke
+			(width 0.153)
+			(type solid)
+		)
+		(layer "F.SilkS")
+	)
+	(gr_line
+		(start 162.56 100.33)
+		(end 165.862 100.33)
+		(stroke
+			(width 0.153)
+			(type solid)
+		)
+		(layer "F.SilkS")
+	)
+	(gr_line
+		(start 165.862 98.298)
+		(end 162.56 98.298)
+		(stroke
+			(width 0.153)
+			(type solid)
+		)
+		(layer "F.SilkS")
+	)
+	(gr_line
+		(start 165.862 94.996)
+		(end 162.56 94.996)
+		(stroke
+			(width 0.153)
+			(type solid)
+		)
+		(layer "F.SilkS")
+	)
+	(gr_line
 		(start 155.575 118.11)
 		(end 155.575 118.745)
@@
 	)
 	(gr_line
+		(start 162.56 101.6)
+		(end 162.56 103.632)
+		(stroke
+			(width 0.153)
+			(type solid)
+		)
+		(layer "F.SilkS")
+	)
+	(gr_line
 		(start 125.73 103.505)
 		(end 125.73 125.095)
@@
 			(width 0.1)
 			(type default)
+		)
+		(layer "F.SilkS")
+	)
+	(gr_line
+		(start 162.56 103.632)
+		(end 165.862 103.632)
+		(stroke
+			(width 0.153)
+			(type solid)
+		)
+		(layer "F.SilkS")
+	)
+	(gr_line
+		(start 162.56 97.028)
+		(end 165.862 97.028)
+		(stroke
+			(width 0.153)
+			(type solid)
 		)
 		(layer "F.SilkS")
@@
 			)
 			(justify left bottom)
+		)
+	)
+	(gr_text "Meltybrain\nControl Board\nv1.0"
+		(at 120.65 96.52 0)
+		(layer "F.SilkS")
+		(effects
+			(font
+				(size 1 1)
+				(thickness 0.2)
+				(bold yes)
+			)
+			(justify left bottom)
