File: controller/silver-platter.kicad_pcb (KiCad board)
At the start: 4 copper layers, 69.9 x 54 mm, 61 parts, among them J1 UART, J11 LED1_B, J12 LED1_G, J13 LED1_R, J14 LED_ANODE, J15 LED2_B, J16 LED2_G, J17 LED2_R, J19 RX_VDD, J2 JTAG/SWJ, J20 iBUS, J21 GND, J22 BOOT, J23 +BATT, J24 -BATT, J3 VDD_ACC, J4 SCL_ACC, J5 SDA_ACC, J6 GND_ACC, J8 CH1_ESC, J9 CH2_ESC, Q1 Q_NMOS, Q2 Q_NMOS, Q3 Q_NMOS, SW1 SW_Push, U1 STM32F205RETx, U2 TLV74033PDBVR, U3 LMR50410Y5FQDBVRQ1

Commit message: Gerbers
Routing:
- net GND: vias 25 -> 39
- added copper zone on B.Cu, net GND
Changed lines of the file:
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@@
+	)
+	(via
+		(at 159.385 88.265)
+		(size 0.6)
+		(drill 0.3)
+		(layers "F.Cu" "B.Cu")
+		(free yes)
+		(net 2)
+	)
+	(via
+		(at 144.78 97.79)
+		(size 0.6)
+		(drill 0.3)
+		(layers "F.Cu" "B.Cu")
+		(free yes)
+		(net 2)
 	)
 	(via
@@
 	)
 	(via
+		(at 169.545 90.805)
+		(size 0.6)
+		(drill 0.3)
+		(layers "F.Cu" "B.Cu")
+		(free yes)
+		(net 2)
+	)
+	(via
+		(at 152.4 88.265)
+		(size 0.6)
+		(drill 0.3)
+		(layers "F.Cu" "B.Cu")
+		(free yes)
+		(net 2)
+	)
+	(via
 		(at 172.212 102.616)
 		(size 0.6)
@@
 	)
 	(via
+		(at 182.88 85.09)
+		(size 0.6)
+		(drill 0.3)
+		(layers "F.Cu" "B.Cu")
+		(free yes)
+		(net 2)
+	)
+	(via
 		(at 142.494 101.145)
 		(size 0.6)
@@
 	)
 	(via
+		(at 137.16 109.855)
+		(size 0.6)
+		(drill 0.3)
+		(layers "F.Cu" "B.Cu")
+		(free yes)
+		(net 2)
+	)
+	(via
 		(at 172.212 96.012)
 		(size 0.6)
@@
 	)
 	(via
+		(at 120.015 99.695)
+		(size 0.6)
+		(drill 0.3)
+		(layers "F.Cu" "B.Cu")
+		(free yes)
+		(net 2)
+	)
+	(via
+		(at 127.635 121.92)
+		(size 0.6)
+		(drill 0.3)
+		(layers "F.Cu" "B.Cu")
+		(free yes)
+		(net 2)
+	)
+	(via
+		(at 166.37 77.47)
+		(size 0.6)
+		(drill 0.3)
+		(layers "F.Cu" "B.Cu")
+		(free yes)
+		(net 2)
+	)
+	(via
 		(at 139.954 107.5425)
 		(size 0.6)
@@
 	)
 	(via
+		(at 172.085 119.38)
+		(size 0.6)
+		(drill 0.3)
+		(layers "F.Cu" "B.Cu")
+		(free yes)
+		(net 2)
+	)
+	(via
+		(at 126.365 89.535)
+		(size 0.6)
+		(drill 0.3)
+		(layers "F.Cu" "B.Cu")
+		(free yes)
+		(net 2)
+	)
+	(via
 		(at 149.606 98.298)
 		(size 0.6)
@@
 	)
 	(via
+		(at 152.4 77.47)
+		(size 0.6)
+		(drill 0.3)
+		(layers "F.Cu" "B.Cu")
+		(free yes)
+		(net 2)
+	)
+	(via
 		(at 131.5455 78.7665)
 		(size 0.6)
@@
 	)
 	(via
+		(at 173.355 111.76)
+		(size 0.6)
+		(drill 0.3)
+		(layers "F.Cu" "B.Cu")
+		(free yes)
+		(net 2)
+	)
+	(via
 		(at 121.92 121.92)
 		(size 0.6)
 		(drill 0.3)
 		(layers "F.Cu" "B.Cu")
+		(net 2)
+	)
+	(via
+		(at 180.34 77.47)
+		(size 0.6)
+		(drill 0.3)
+		(layers "F.Cu" "B.Cu")
+		(free yes)
 		(net 2)
 	)
@@
 		(layer "F.Cu")
 		(hatch edge 0.5)
-		(priority 1)
+		(priority 2)
 		(connect_pads yes
 			(clearance 0.1)
@@
 			)
 		)
+	)
+	(zone
+		(net 2)
+		(net_name "GND")
+		(layer "F.Cu")
+		(hatch edge 0.5)
+		(priority 1)
+		(connect_pads no
+			(clearance 1)
+		)
+		(min_thickness 0.5)
+		(filled_areas_thickness no)
+		(fill yes
+			(thermal_gap 0.5)
+			(thermal_bridge_width 0.5)
+		)
+		(polygon
+			(pts
+				(xy 118.11 73.025) (xy 187.96 73.025) (xy 187.96 127) (xy 118.11 127)
+			)
+		)
+	)
+	(zone
+		(net 2)
+		(net_name "GND")
+		(layer "B.Cu")
+		(hatch edge 0.5)
+		(priority 1)
+		(connect_pads no
+			(clearance 1)
+		)
+		(min_thickness 0.5)
+		(filled_areas_thickness no)
+		(fill yes
+			(thermal_gap 0.5)
+			(thermal_bridge_width 0.5)
+		)
+		(polygon
+			(pts
+				(xy 118.11 73.025) (xy 187.96 73.025) (xy 187.96 127) (xy 118.11 127)
+			)
+		)
